Commit message: Got custom plugin working to control arm via ros2_control

File: hitw_description/urdf/hitw_arm.urdf.xacro (robot description, xacro)
@@ -16,5 +16,5 @@
       </visual>
     </link>
-    <link name="${prefix}arm_link_1">
+    <link name="${prefix}link1">
       <visual>
         <origin xyz="0 0 0.25"/>
@@ -25,5 +25,5 @@
       </visual>
     </link>
-    <link name="${prefix}arm_link_2">
+    <link name="${prefix}link2">
       <visual>
         <origin xyz="0 0 0.25"/>
@@ -34,17 +34,17 @@
       </visual>
     </link>
-    <joint name="${prefix}arm_joint_1" type="revolute">
+    <joint name="${prefix}joint1" type="revolute">
       <axis xyz="0 1 0"/>
       <limit effort="1000.0" lower="-1.5708" upper="1.5708" velocity="0.5"/>
       <origin rpy="0 0 0" xyz="0 0 0"/>
       <parent link="${prefix}base_link"/>
-      <child link="${prefix}arm_link_1"/>
+      <child link="${prefix}link1"/>
     </joint>
-    <joint name="${prefix}arm_joint_2" type="revolute">
+    <joint name="${prefix}joint2" type="revolute">
       <axis xyz="0 1 0"/>
       <limit effort="1000.0" lower="-1.5708" upper="1.5708" velocity="0.5"/>
       <origin rpy="0 0 0" xyz="0 0 0.5"/>
-      <parent link="${prefix}arm_link_1"/>
-      <child link="${prefix}arm_link_2"/>
+      <parent link="${prefix}link1"/>
+      <child link="${prefix}link2"/>
     </joint>
   </xacro:macro>

File: hitw_description/urdf/ros2_control.xacro (robot description, xacro)
@@ -2,9 +2,10 @@
 <robot xmlns:xacro="http://www.ros.org/wiki/xacro">
   <xacro:macro name="hitw_arm_ros2_control" params="prefix">
-    <ros2_control name="GazeboSystem" type="system">
+    <ros2_control name="HITWBot" type="system">
       <hardware>
-        <plugin>gazebo_ros2_control/GazeboSystem</plugin>
+        <plugin>hitw_hardware/HITWBotSystemPositionOnlyHardware</plugin>
+        <param name="hw_slowdown">100</param>
       </hardware>
-      <joint name="${prefix}arm_joint_1">
+      <joint name="${prefix}joint1">
         <command_interface name="position">
           <param name="min">-1</param>
@@ -12,7 +13,7 @@
         </command_interface>
         <state_interface name="position"/>
-        <state_interface name="velocity"/>
+        <!--<state_interface name="velocity"/>-->
       </joint>
-      <joint name="${prefix}arm_joint_2">
+      <joint name="${prefix}joint2">
         <command_interface name="position">
           <param name="min">-1</param>
@@ -20,14 +21,16 @@
         </command_interface>
         <state_interface name="position"/>
-        <state_interface name="velocity"/>
+        <!--<state_interface name="velocity"/>-->
       </joint>
     </ros2_control>
+    <!--
     <gazebo>
       <plugin name="gazebo_ros2_control" filename="libgazebo_ros2_control.so">
         <robotNamespace>/hitw</robotNamespace>
         <robotParam>/robot_description</robotParam>
-        <parameters>$(find hitw_description)/config/my_controllers.yaml</parameters>
+        <parameters>$(find hitw_controllers)/config/my_controllers.yaml</parameters>
       </plugin>
     </gazebo>
+    -->
   </xacro:macro>
 </robot>

File: hitw_description/urdf/transmissions.xacro (robot description, xacro)
@@ -2,20 +2,20 @@
 <robot xmlns:xacro="http://www.ros.org/wiki/xacro" >
   <xacro:macro name="hitw_arm_transmissions" params="prefix">
-    <transmission name="${prefix}transmission_1">
+    <transmission name="${prefix}transmission1">
       <type>transmission_interface/SimpleTransmission</type>
-      <joint name="${prefix}arm_joint_1">
+      <joint name="${prefix}joint1">
         <hardwareInterface>EffortJointInterface</hardwareInterface>
       </joint>
-      <actuator name="${prefix}arm_motor_1">
+      <actuator name="${prefix}motor1">
         <hardwareInterface>EffortJointInterface</hardwareInterface>
         <mechanicalReduction>1</mechanicalReduction>
       </actuator>
     </transmission>
-    <transmission name="${prefix}transmission_2">
+    <transmission name="${prefix}transmission2">
       <type>transmission_interface/SimpleTransmission</type>
-      <joint name="${prefix}arm_joint_2">
+      <joint name="${prefix}joint_2">
         <hardwareInterface>EffortJointInterface</hardwareInterface>
       </joint>
-      <actuator name="${prefix}arm_motor_2">
+      <actuator name="${prefix}motor2">
         <hardwareInterface>EffortJointInterface</hardwareInterface>
         <mechanicalReduction>1</mechanicalReduction>
