Commit message: Adding Gazebo functionality (in progress)

File: hitw_description/urdf/hitw_arm_macro.urdf.xacro (robot description, xacro)
@@ -8,4 +8,5 @@
   <xacro:include filename="transmissions.xacro" />
   <xacro:include filename="materials.xacro" />
+  <xacro:include filename="camera.xacro" />
   <!-- Used for fixing robot -->
   <link name="world"/>
@@ -13,4 +14,5 @@
     <origin xyz="0 0 0" rpy="0 0 0" />
   </xacro:hitw_arm>
+  <xacro:hitw_camera prefix="$(arg prefix)" />
   <xacro:hitw_arm_ros2_control prefix="$(arg prefix)" />
   <xacro:hitw_arm_transmissions prefix="$(arg prefix)" />

File: hitw_description/urdf/materials.xacro (robot description, xacro)
@@ -3,4 +3,7 @@
   <material name="blue">
     <color rgba="0 0 0.8 1"/>
+  </material>
+  <material name="red">
+    <color rgba="0.8 0 0 1"/>
   </material>
   <material name="black">
