Commit message: Arm now visible in gazebo, still having trouble controlling it

File: hitw_description/urdf/camera.xacro (robot description, xacro)
@@ -1,4 +1,4 @@
 <?xml version="1.0"?>
-<robot xmlns:xacro="http://www.ros.org/wiki/xacro" >
+<robot xmlns:xacro="http://www.ros.org/wiki/xacro">
   <xacro:macro name="hitw_camera" params="prefix">
     <link name="${prefix}rgb_camera_link">

File: hitw_description/urdf/hitw_arm.urdf.xacro (robot description, xacro)
@@ -1,10 +1,13 @@
 <?xml version="1.0"?>
-<robot xmlns:xacro="http://www.ros.org/wiki/xacro" >
+<robot xmlns:xacro="http://www.ros.org/wiki/xacro">
   <xacro:macro name="hitw_arm" params="parent prefix *origin">
+    <xacro:include filename="inertia_macro.xacro"/>
+    <!--********************************* BASE JOINT *********************************-->
     <joint name="${prefix}base_joint" type="fixed">
-      <xacro:insert_block name="origin" />
+      <xacro:insert_block name="origin"/>
       <parent link="${parent}"/>
-      <child link="${prefix}base_link" />
+      <child link="${prefix}base_link"/>
     </joint>
+    <!--********************************* BASE LINK *********************************-->
     <link name="${prefix}base_link">
       <visual>
@@ -15,5 +18,16 @@
         <material name="black"/>
       </visual>
+      <collision>
+        <origin xyz="0 0 0.05"/>
+        <geometry>
+          <cylinder radius="0.25" length="0.1"/>
+        </geometry>
+      </collision>
+      <xacro:cylinder_inertia m="0.5" r="0.25" h="0.1"/>
     </link>
+    <gazebo reference="${prefix}base_link">
+      <material>Gazebo/Black</material>
+    </gazebo>
+    <!--********************************* LINK 1 *********************************-->
     <link name="${prefix}link1">
       <visual>
@@ -24,5 +38,20 @@
         <material name="white"/>
       </visual>
+      <collision>
+        <origin xyz="0 0 0.25"/>
+        <geometry>
+          <box size="0.1 0.1 0.5"/>
+        </geometry>
+      </collision>
+      <xacro:box_inertia m="0.5" d="0.1" w="0.1" h="0.5"/>
     </link>
+    <gazebo reference="${prefix}link1">
+      <material>Gazebo/White</material>
+      <kp>100000.0</kp>
+      <kd>1.0</kd>
+      <mu1>10.0</mu1>
+      <mu2>10.0</mu2>
+    </gazebo>
+    <!--********************************* LINK 2 *********************************-->
     <link name="${prefix}link2">
       <visual>
@@ -33,5 +62,20 @@
         <material name="blue"/>
       </visual>
+      <collision>
+        <origin xyz="0 0 0.25"/>
+        <geometry>
+          <box size="0.1 0.1 0.5"/>
+        </geometry>
+      </collision>
+      <xacro:box_inertia m="0.5" d="0.1" w="0.1" h="0.5"/>
     </link>
+    <gazebo reference="${prefix}link2">
+      <material>Gazebo/Blue</material>
+      <kp>100000.0</kp>
+      <kd>1.0</kd>
+      <mu1>10.0</mu1>
+      <mu2>10.0</mu2>
+    </gazebo>
+    <!--********************************* JOINT 1 *********************************-->
     <joint name="${prefix}joint1" type="revolute">
       <axis xyz="0 1 0"/>
@@ -40,5 +84,9 @@
       <parent link="${prefix}base_link"/>
       <child link="${prefix}link1"/>
+      <limit
+        lower="${-2.0*pi}"
+        upper="${2.0*pi}"/>
     </joint>
+    <!--********************************* JOINT 2 *********************************-->
     <joint name="${prefix}joint2" type="revolute">
       <axis xyz="0 1 0"/>
@@ -47,4 +95,7 @@
       <parent link="${prefix}link1"/>
       <child link="${prefix}link2"/>
+      <limit
+        lower="${-2.0*pi}"
+        upper="${2.0*pi}"/>
     </joint>
   </xacro:macro>

File: hitw_description/urdf/hitw_arm_macro.urdf.xacro (robot description, xacro)
@@ -1,19 +1,19 @@
 <?xml version="1.0"?>
 <robot xmlns:xacro="http://www.ros.org/wiki/xacro" name="hitw_arm_robot">
-  <xacro:arg name="prefix" default="" />
+  <xacro:arg name="prefix" default=""/>
   <!-- Import hitw_arm macro -->
-  <xacro:include filename="hitw_arm.urdf.xacro" />
+  <xacro:include filename="hitw_arm.urdf.xacro"/>
   <!-- Import ros2_control paramaters-->
-  <xacro:include filename="ros2_control.xacro" />
-  <xacro:include filename="transmissions.xacro" />
-  <xacro:include filename="materials.xacro" />
-  <xacro:include filename="camera.xacro" />
+  <xacro:include filename="ros2_control.xacro"/>
+  <xacro:include filename="transmissions.xacro"/>
+  <xacro:include filename="materials.xacro"/>
+  <xacro:include filename="camera.xacro"/>
   <!-- Used for fixing robot -->
   <link name="world"/>
   <xacro:hitw_arm parent="world" prefix="$(arg prefix)">
-    <origin xyz="0 0 0" rpy="0 0 0" />
+    <origin xyz="0 0 0" rpy="0 0 0"/>
   </xacro:hitw_arm>
-  <xacro:hitw_camera prefix="$(arg prefix)" />
-  <xacro:hitw_arm_ros2_control prefix="$(arg prefix)" />
-  <xacro:hitw_arm_transmissions prefix="$(arg prefix)" />
+  <xacro:hitw_camera prefix="$(arg prefix)"/>
+  <xacro:hitw_arm_ros2_control prefix="$(arg prefix)"/>
+  <xacro:hitw_arm_transmissions prefix="$(arg prefix)"/>
 </robot>

File: hitw_description/urdf/materials.xacro (robot description, xacro)
@@ -1,4 +1,4 @@
 <?xml version="1.0"?>
-<robot xmlns:xacro="http://www.ros.org/wiki/xacro" >
+<robot xmlns:xacro="http://www.ros.org/wiki/xacro">
   <material name="blue">
     <color rgba="0 0 0.8 1"/>

File: hitw_description/urdf/transmissions.xacro (robot description, xacro)
@@ -1,4 +1,4 @@
 <?xml version="1.0"?>
-<robot xmlns:xacro="http://www.ros.org/wiki/xacro" >
+<robot xmlns:xacro="http://www.ros.org/wiki/xacro">
   <xacro:macro name="hitw_arm_transmissions" params="prefix">
     <transmission name="${prefix}transmission1">
@@ -14,5 +14,5 @@
     <transmission name="${prefix}transmission2">
       <type>transmission_interface/SimpleTransmission</type>
-      <joint name="${prefix}joint_2">
+      <joint name="${prefix}joint2">
         <hardwareInterface>EffortJointInterface</hardwareInterface>
       </joint>

Commit message: Gazebo simulation working except for camera

File: hitw_description/urdf/camera.xacro (robot description, xacro)
@@ -11,4 +11,7 @@
       </visual>
     </link>
+    <gazebo reference="${prefix}rgb_camera_link">
+      <material>Gazebo/Black</material>
+    </gazebo>
     <joint name="${prefix}rgb_camera_link_joint" type="fixed">
       <origin rpy="0 0 0" xyz="1.0 0.0 0.5"/>

File: hitw_description/urdf/hitw_arm.urdf.xacro (robot description, xacro)
@@ -1,12 +1,6 @@
 <?xml version="1.0"?>
 <robot xmlns:xacro="http://www.ros.org/wiki/xacro">
-  <xacro:macro name="hitw_arm" params="parent prefix *origin">
+  <xacro:macro name="hitw_arm_core" params="parent prefix *origin">
     <xacro:include filename="inertia_macro.xacro"/>
-    <!--********************************* BASE JOINT *********************************-->
-    <joint name="${prefix}base_joint" type="fixed">
-      <xacro:insert_block name="origin"/>
-      <parent link="${parent}"/>
-      <child link="${prefix}base_link"/>
-    </joint>
     <!--********************************* BASE LINK *********************************-->
     <link name="${prefix}base_link">
@@ -29,4 +23,10 @@
       <material>Gazebo/Black</material>
     </gazebo>
+    <!--********************************* BASE JOINT *********************************-->
+    <joint name="${prefix}base_joint" type="fixed">
+      <xacro:insert_block name="origin"/>
+      <parent link="${parent}"/>
+      <child link="${prefix}base_link"/>
+    </joint>
     <!--********************************* LINK 1 *********************************-->
     <link name="${prefix}link1">
@@ -48,8 +48,4 @@
     <gazebo reference="${prefix}link1">
       <material>Gazebo/White</material>
-      <kp>100000.0</kp>
-      <kd>1.0</kd>
-      <mu1>10.0</mu1>
-      <mu2>10.0</mu2>
     </gazebo>
     <!--********************************* LINK 2 *********************************-->
@@ -72,8 +68,4 @@
     <gazebo reference="${prefix}link2">
       <material>Gazebo/Blue</material>
-      <kp>100000.0</kp>
-      <kd>1.0</kd>
-      <mu1>10.0</mu1>
-      <mu2>10.0</mu2>
     </gazebo>
     <!--********************************* JOINT 1 *********************************-->

File: hitw_description/urdf/hitw_arm_macro.urdf.xacro (robot description, xacro)
@@ -2,4 +2,5 @@
 <robot xmlns:xacro="http://www.ros.org/wiki/xacro" name="hitw_arm_robot">
   <xacro:arg name="prefix" default=""/>
+  <xacro:arg name="use_gazebo" default="false"/>
   <!-- Import hitw_arm macro -->
   <xacro:include filename="hitw_arm.urdf.xacro"/>
@@ -11,9 +12,9 @@
   <!-- Used for fixing robot -->
   <link name="world"/>
-  <xacro:hitw_arm parent="world" prefix="$(arg prefix)">
+  <xacro:hitw_arm_core parent="world" prefix="$(arg prefix)">
     <origin xyz="0 0 0" rpy="0 0 0"/>
-  </xacro:hitw_arm>
+  </xacro:hitw_arm_core>
   <xacro:hitw_camera prefix="$(arg prefix)"/>
-  <xacro:hitw_arm_ros2_control prefix="$(arg prefix)"/>
+  <xacro:hitw_arm_ros2_control prefix="$(arg prefix)" use_gazebo="$(arg use_gazebo)"/>
   <xacro:hitw_arm_transmissions prefix="$(arg prefix)"/>
 </robot>

File: hitw_description/urdf/ros2_control.xacro (robot description, xacro)
@@ -1,36 +1,53 @@
 <?xml version="1.0"?>
 <robot xmlns:xacro="http://www.ros.org/wiki/xacro">
-  <xacro:macro name="hitw_arm_ros2_control" params="prefix">
-    <ros2_control name="HITWBot" type="system">
-      <hardware>
-        <plugin>hitw_hardware/HITWBotSystemPositionOnlyHardware</plugin>
-        <param name="hw_slowdown">100</param>
-      </hardware>
-      <joint name="${prefix}joint1">
-        <command_interface name="position">
-          <param name="min">-1</param>
-          <param name="max">1</param>
-        </command_interface>
-        <state_interface name="position"/>
-        <!--<state_interface name="velocity"/>-->
-      </joint>
-      <joint name="${prefix}joint2">
-        <command_interface name="position">
-          <param name="min">-1</param>
-          <param name="max">1</param>
-        </command_interface>
-        <state_interface name="position"/>
-        <!--<state_interface name="velocity"/>-->
-      </joint>
-    </ros2_control>
-    <!--
-    <gazebo>
-      <plugin name="gazebo_ros2_control" filename="libgazebo_ros2_control.so">
-        <robotNamespace>/hitw</robotNamespace>
-        <robotParam>/robot_description</robotParam>
-        <parameters>$(find hitw_controllers)/config/my_controllers.yaml</parameters>
-      </plugin>
-    </gazebo>
-    -->
+  <xacro:macro name="hitw_arm_ros2_control" params="prefix use_gazebo">
+    <xacro:if value="${not use_gazebo}">
+      <ros2_control name="HITWBot" type="system">
+        <hardware>
+          <plugin>hitw_hardware/HITWBotSystemPositionOnlyHardware</plugin>
+          <param name="hw_slowdown">100</param>
+        </hardware>
+        <joint name="${prefix}joint1">
+          <command_interface name="position">
+            <param name="min">-1</param>
+            <param name="max">1</param>
+          </command_interface>
+          <state_interface name="position"/>
+        </joint>
+        <joint name="${prefix}joint2">
+          <command_interface name="position">
+            <param name="min">-1</param>
+            <param name="max">1</param>
+          </command_interface>
+          <state_interface name="position"/>
+        </joint>
+      </ros2_control>
+    </xacro:if>
+    <xacro:if value="${use_gazebo}">
+      <ros2_control name="GazeboSystem" type="system">
+        <hardware>
+          <plugin>gazebo_ros2_control/GazeboSystem</plugin>
+        </hardware>
+        <joint name="${prefix}joint1">
+          <command_interface name="position">
+            <param name="min">-6.283185307179586</param>
+            <param name="max">6.283185307179586</param>
+          </command_interface>
+          <state_interface name="position"/>
+        </joint>
+        <joint name="${prefix}joint2">
+          <command_interface name="position">
+            <param name="min">-6.283185307179586</param>
+            <param name="max">6.283185307179586</param>
+          </command_interface>
+          <state_interface name="position"/>
+        </joint>
+      </ros2_control>
+      <gazebo>
+        <plugin name="gazebo_ros2_control" filename="libgazebo_ros2_control.so">
+          <parameters>$(find hitw_controllers)/config/gazebo_controllers.yaml</parameters>
+        </plugin>
+      </gazebo>
+    </xacro:if>
   </xacro:macro>
 </robot>

Commit message: Updated camera positioning URDF

File: hitw_description/urdf/camera.xacro (robot description, xacro)
@@ -4,5 +4,5 @@
     <link name="${prefix}rgb_camera_link">
       <visual>
-        <origin xyz="1 0 1"/>
+        <origin xyz="0 0 0"/>
         <geometry>
           <box size="0.05 0.05 0.05"/>
@@ -15,5 +15,5 @@
     </gazebo>
     <joint name="${prefix}rgb_camera_link_joint" type="fixed">
-      <origin rpy="0 0 0" xyz="1.0 0.0 0.5"/>
+      <origin rpy="0 0 ${pi/2}" xyz="0.0 1.0 0.5"/>
 	  <parent link="${prefix}base_link"/>
 	  <child link="${prefix}rgb_camera_link"/>
